Commit message: tue r5cop

File: x80sv_description/urdf/wheel.xacro (robot description, xacro)
@@ -5,7 +5,7 @@
     xmlns:controller="http://playerstage.sourceforge.net/gazebo/xmlschema/#controller"
     xmlns:interface="http://playerstage.sourceforge.net/gazebo/xmlschema/#interface">
-    <macro name="wheel" params="suffix parent *origin">
+    <xacro:macro name="wheel" params="suffix parent *origin">
         <joint name="${parent}_${suffix}_wheel_joint" type="continuous">
-            <insert_block name="origin" />
+            <xacro:insert_block name="origin" />
             <axis xyz="0 1 0" />
             <anchor xyz="0 0 0" />
@@ -50,4 +50,4 @@
             <mechanicalReduction>1.0</mechanicalReduction>
         </transmission>
-    </macro>
+    </xacro:macro>
 </robot>
